File: shifr_pcb/shifr_pcb.kicad_pcb (KiCad board)
At the start: 2 copper layers, 191 x 101 mm, 93 parts, among them SW1 Power Switch, SW2 Reset Switch, U1 Nice_Nano_V2

Commit message: Alternate silkscreen
Other:
- board text added: "WayWayWay"
- board text added: "github.com/CityRunner/shifr-keyboard"
- board text added: "v1.4"
- board text removed: "JLCJLCJLCJLC"
- board text removed: "https://github.com/CityRunner/shifr"
- board text removed: "v1.3"

Commit message: Changed power switch footprint
Connections:
- U1 pad 3: unconnected-(U1-GND-Pad3) -> ground
- U1 pad 4: unconnected-(U1-GND-Pad4) -> ground

Commit message: update main pcb
Parts:
- removed H1, H2, H3, H4, H5: MountingHole, MountingHole:MountingHole_2.2mm_M2_Pad_Via
- removed H6, H7, H8, H9: MountingHole, MountingHole:MountingHole_2.2mm_M2_ISO14580
- added REF**: MountingHole_2.2mm_M2_ISO14580, MountingHole:MountingHole_2.2mm_M2_ISO14580, F.Cu at (181.2, 58.8)
- added REF**: MountingHole_2.2mm_M2_Pad_Via, MountingHole:MountingHole_2.2mm_M2_Pad_Via, F.Cu at (59.0, 64.0)
- added REF**: MountingHole_2.2mm_M2_ISO14580, MountingHole:MountingHole_2.2mm_M2_ISO14580, F.Cu at (181.2, 44.8)
- added REF**: MountingHole_2.2mm_M2_ISO14580, MountingHole:MountingHole_2.2mm_M2_ISO14580, F.Cu at (207.2, 58.8)
- added REF**: MountingHole_2.2mm_M2_Pad_Via, MountingHole:MountingHole_2.2mm_M2_Pad_Via, F.Cu at (135.0, 102.0)
- added REF**: MountingHole_2.2mm_M2_Pad_Via, MountingHole:MountingHole_2.2mm_M2_Pad_Via, F.Cu at (211.0, 121.0)
- added REF**: MountingHole_2.2mm_M2_Pad_Via, MountingHole:MountingHole_2.2mm_M2_Pad_Via, F.Cu at (59.0, 121.0)
- added REF**: MountingHole_2.2mm_M2_ISO14580, MountingHole:MountingHole_2.2mm_M2_ISO14580, F.Cu at (207.2, 44.8)
- added REF**: MountingHole_2.2mm_M2_Pad_Via, MountingHole:MountingHole_2.2mm_M2_Pad_Via, F.Cu at (211.0, 64.0)
